File: Diode Sallen-Key VCF.kicad_sch (KiCad schematic)
At the start: 98 parts, among them J1 V/Oct CV, J10 Conn_02x05_Odd_Even, J11 Conn_01x01, J12 Conn_01x01, J13 Conn_01x01, J14 Conn_01x01, J15 Conn_01x01, J16 Conn_01x01, J17 Conn_01x01, J18 Conn_01x01, J19 Conn_01x01, J2 CV, J20 Conn_01x01, J21 Out, J3 In, J4 Conn_01x01, J5 Conn_01x01, J6 Conn_01x01, J7 Conn_01x01, J8 Conn_01x01, J9 Conn_01x01, SW1 SW_Rotary_4x3, U1 TL072, U2 TL072, U3 TL072, U4 TL072, U5 TL072, U6 TL072, U7 TL072

Commit message: Quad opamps
Parts:
- removed C17, C18, C6, C7: 0.1u, Capacitor_THT:C_Disc_D5.1mm_W3.2mm_P5.00mm, symbol Device:C
- removed U1, U2, U6, U7: TL072, Package_DIP:DIP-8_W7.62mm_Socket, symbol Amplifier_Operational:TL072
- added U1, U8: TL074, Package_DIP:DIP-14_W7.62mm_Socket, symbol Amplifier_Operational:TL074
Connections:
- net CV_IN: now also U8.12 (+)
- net GND: now also U1.3 (+), U8.5 (+)
- net IN_BUF: now also U8.1, U8.2 (-)
- net IN_INV: now also U8.7
- net OUT_BUF: now also U1.8, U1.9 (-)
- net RES_WIPER: now also U1.12 (+)
- net VCC: now also U1.4 (V+), U8.4 (V+)
- net VEE: now also U1.11 (V-), U8.11 (V-)
- net VOCT_IN: now also U8.10 (+)
- net at D7.2 (A), D8.1 (K), R25.2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: now also U1.2 (-)
- net at D7.1 (K), D8.2 (A), RV6.1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: now also U1.1
- net at R9.1: now also U8.13 (-), U8.14
- net at C1.2, D4.1 (K), D5.2 (A): now also U1.10 (+)
- net at RV7.1, RV7.2: now also U1.13 (-), U1.14
- net at R21.2: now also U1.6 (-), U1.7
- net at R3.2, R5.2: now also U8.3 (+)
- net at R25.1, RV6.3: now also U1.5 (+)
- net at RV5.3: now also U8.8, U8.9 (-)
- net at R10.1, R12.2: now also U8.6 (-)
Other:
- moved on the sheet: C20, C21, C4, C5, U3C, U4C, U5C

Commit message: small tweaks
Parts:
- R1: value 100k -> 1M
- renumbered C12 to C10, C13 to C11, C14 to C12, C15 to C13, C16 to C14, C20 to C15, C21 to C16, C19 to C17, C8 to C6, C9 to C7, C10 to C8, C11 to C9, R26 to R25, R25 to R26, U8 to U1, U3 to U2, U4 to U3, U5 to U4, U1 to U5
Other:
- moved on the sheet: C1, C10, C11, C12, C13, C14, C15, C16, C17, C2, C3, C4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

Commit message: small tweaks
Parts:
- added R2: 12k, Resistor_THT:R_Axial_DIN0207_L6.3mm_D2.5mm_P10.16mm_Horizontal, symbol Device:R
- RV1: value 50k lin -> 50k
- RV2: value 10k lin -> 10k
- RV3: value 20k log -> 100k
- renumbered R8 to R10, R10 to R11, R11 to R12, R12 to R13, R13 to R14, R14 to R15, R15 to R16, R16 to R17, R17 to R18, R18 to R19, R19 to R20, R20 to R21, R21 to R22, R22 to R23, R23 to R24, R24 to R25, R25 to R26, R26 to R27, R27 to R28, R28 to R29, R2 to R3, R3 to R4, R4 to R5, R5 to R6, R9 to R7, R6 to R8, R7 to R9
Connections:
- net AUDIO_IN: now also R2.2
- net GND: now also R2.1
Other:
- moved on the sheet: R29, R4, R7, U5A

Commit message: missed output resistor
Parts:
- added R30: 1k, Resistor_THT:R_Axial_DIN0207_L6.3mm_D2.5mm_P10.16mm_Horizontal, symbol Device:R
- C17: value 10p -> 22p
Connections:
- net AUDIO_OUT: now also R30.2; no longer C17.2, R28.2, U4.7
- new net: C17.2, R28.2, R30.1, U4.7
Changed lines of the file:
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@@
 	(wire
 		(pts
+			(xy 322.58 81.28) (xy 388.62 81.28)
+		)
+		(stroke
+			(width 0)
+			(type default)
+		)
+	)
+	(wire
+		(pts
 			(xy 137.16 173.99) (xy 165.1 173.99)
 		)
@@
 	(wire
 		(pts
-			(xy 308.61 81.28) (xy 388.62 81.28)
+			(xy 308.61 81.28) (xy 314.96 81.28)
 		)
 		(stroke
@@
 	)
 	(label "AUDIO_OUT"
-		(at 312.42 81.28 0)
+		(at 346.71 81.28 0)
 		(effects
 			(font
@@
 			)
 		)
-		(property "Value" "10p"
+		(property "Value" "22p"
 			(at 295.91 100.33 90)
 			(show_name no)
@@
 					(unit 1)
 				)
+			)
+		)
+	)
+	(symbol
+		(lib_id "Device:R")
+		(at 318.77 81.28 90)
+		(unit 1)
+		(body_style 1)
+		(exclude_from_sim no)
+		(in_bom yes)
+		(on_board yes)
+		(in_pos_files yes)
+		(dnp no)
+		(fields_autoplaced yes)
+		(property "Reference" "R30"
+			(at 318.77 74.93 90)
+			(show_name no)
+			(do_not_autoplace no)
+			(effects
+				(font
+					(size 1.27 1.27)
+				)
+			)
+		)
+		(property "Value" "1k"
+			(at 318.77 77.47 90)
+			(show_name no)
+			(do_not_autoplace no)
+			(effects
+				(font
+					(size 1.27 1.27)
+				)
+			)
+		)
+		(property "Footprint" "Resistor_THT:R_Axial_DIN0207_L6.3mm_D2.5mm_P10.16mm_Horizontal"
+			(at 318.77 83.058 90)
+			(hide yes)
+			(show_name no)
+			(do_not_autoplace no)
+			(effects
+				(font
+					(size 1.27 1.27)
+				)
+			)
+		)
+		(property "Datasheet" ""
+			(at 318.77 81.28 0)
+			(hide yes)
+			(show_name no)
+			(do_not_autoplace no)
+			(effects
+				(font
+					(size 1.27 1.27)
+				)
+			)
+		)
+		(property "Description" "Resistor"
+			(at 318.77 81.28 0)
+			(hide yes)
+			(show_name no)
+			(do_not_autoplace no)
+			(effects
+				(font
+					(size 1.27 1.27)
+				)
+			)
+		)
+		(pin "2"
+		)
+		(pin "1"
+		)
+		(instances
+			(project "Diode Sallen-Key VCF"
+				(path "/044ce31f-a56b-4ee2-9d5d-adcdbf76b311"
+					(reference "R30")
+					(unit 1)
+				)
